Commit message: Fixed relative grasps.

File: models/fork.urdf (robot description, URDF)
Before this commit: robot fork, 1 links, 0 joints
Links:
- link base_link: geometry collision mesh filename=fork.stl scale=0.01 0.01 0.01; visual mesh filename=fork.stl scale=0.01 0.01 0.01

File: models/knife.urdf (robot description, URDF)
Before this commit: robot fork, 1 links, 0 joints
Links:
- link base_link: geometry collision mesh filename=knife.stl scale=0.01 0.01 0.01; visual mesh filename=knife.stl scale=0.01 0.01 0.01

File: models/spoon.urdf (robot description, URDF)
Before this commit: robot fork, 1 links, 0 joints
Links:
- link base_link: geometry collision mesh filename=spoon.stl scale=0.01 0.01 0.01; visual mesh filename=spoon.stl scale=0.01 0.01 0.01
