Commit message: Working on collision checking between objects.

File: models/plate.urdf (robot description, URDF)
Before this commit: robot fork, 1 links, 0 joints
Links:
- link base_link: geometry collision mesh filename=bowl.stl scale=0.001 0.001 0.001; visual mesh filename=bowl.stl scale=0.001 0.001 0.001

File: models/short_floor.urdf (robot description, URDF)
Before this commit: robot flat_terrain, 1 links, 0 joints
Links:
- link base_link: geometry collision box size=1.23 1.54 0.1; visual box size=1.23 1.54 0.1

Commit message: Changed bowl model to obj

File: models/plate.urdf (robot description, URDF)
Before this commit: robot fork, 1 links, 0 joints
Links:
- link base_link: geometry collision mesh filename=bowl.obj scale=0.001 0.001 0.001; visual mesh filename=bowl.obj scale=0.001 0.001 0.001

Commit message: Fixed Bowl model

File: models/plate.urdf (robot description, URDF)
Before this commit: robot fork, 1 links, 0 joints
Links:
- link base_link: geometry collision mesh filename=new_bowl.obj scale=1 1 1; visual mesh filename=new_bowl.obj scale=1 1 1

File: models/short_floor.urdf (robot description, URDF)
Before this commit: robot flat_terrain, 1 links, 0 joints
Links:
- link base_link: geometry collision box size=1.524 1.2192 0.1; visual box size=1.524 1.2192 0.1
