Commit message: Working TAMP Door Opening

File: models/block.urdf (robot description, URDF)
Before this commit: robot block, 1 links, 0 joints
Links:
- link base_link: geometry collision box size=0.05 0.05 0.05; visual box size=0.05 0.05 0.05

Commit message: Testing Spring

File: models/block.urdf (robot description, URDF)
Before this commit: robot block, 1 links, 0 joints
Links:
- link base_link: geometry collision box size=0.05 0.05 0.11; visual box size=0.05 0.05 0.11
