Commit message: Working on Door Opening

File: models/door.urdf (robot description, URDF)
Before this commit: robot urdf_door, 3 links, 2 joints
Links:
- added link door_knob, mass .0; collision box size=0.07 0.05 0.05; visual box size=0.05 0.07 0.05
Joints:
- added joint knob_door: type fixed, parent childA, child door_knob, origin xyz=0.75 0.07 0.425

Commit message: Working on Door Traj

File: models/door.urdf (robot description, URDF)
Before this commit: robot urdf_door, 4 links, 3 joints
Links:
- removed link door_knob
- added link knob, mass .0; collision box size=0.07 0.05 0.05; visual box size=0.05 0.07 0.05
Joints:
- joint knob_door: child door_knob -> knob

Commit message: Door Traj Done.

File: models/door.urdf (robot description, URDF)
Before this commit: robot urdf_door, 4 links, 3 joints
Links:
- link knob: geometry collision box size=0.05 0.07 0.05; visual box size=0.05 0.07 0.05

Commit message: Working on Wrench Transform and Testing Door.

File: models/door.urdf (robot description, URDF)
Before this commit: robot urdf_door, 4 links, 3 joints
Links:
- link knob: geometry collision box size=0.05 0.20 0.05; visual box size=0.05 0.20 0.05
Joints:
- joint knob_door: origin xyz=0.75 0.07 0.425 -> xyz=0.75 0 0.425
